File: pcb/mini_line_mixer.kicad_sch (KiCad schematic)
At the start: 89 parts, among them J1 Ach1, J10 B Out, J101 Center -, J11 Phone Out, J2 Ach2, J3 Ach3, J4 A/Bch4, J5 Bch1, J6 Bch2, J7 Bch3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

Commit message: Fixed parts discription
Parts:
- C1, C103, C11, C14, C2, C3, C4, C5, C6, C7, C8: Part Model No. サイズ max 5phi x 11mmまで -> サイズ max 5phi x 11mm
- RV11: Part Model No. ALPS RK09L1240-F15-C0-B503(2連) -> ALPS RK09L1240-F15-C0-B503 2gang (2連)
- RV4: Part Model No. ALPS RK09L1240-F15-C0-A103(2連) -> ALPS RK09L1240-F15-C0-A103 2gang (2連)
- SW101: Part Model No. NKK B-12CCPRM -> NKK B-12CCPR
- U1, U2, U3: symbol Amplifier_Operational:NJM4580 -> Amplifier_Operational:NJM5532
Changed lines of the file:
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@@
       (effects (font (size 1.27 1.27)) hide)
     )
-    (property "Part Model No." "サイズ max 5phi x 11mmまで" (id 4) (at 40.005 186.055 0)
+    (property "Part Model No." "サイズ max 5phi x 11mm" (id 4) (at 40.005 186.055 0)
       (effects (font (size 1.27 1.27)) hide)
     )
@@
     (pin "1")
   )
-  (symbol (lib_id "Amplifier_Operational:NJM4580") (at 124.46 27.94 0) (unit 3)
+  (symbol (lib_id "Amplifier_Operational:NJM5532") (at 124.46 27.94 0) (unit 3)
     (in_bom yes) (on_board yes)
     (property "Reference" "U1" (id 0) (at 123.444 26.6699 0)
@@
       (effects (font (size 1.27 1.27)) hide)
     )
-    (property "Datasheet" "http://www.njr.com/semicon/PDF/NJM4580_E.pdf" (id 3) (at 124.46 27.94 0)
+    (property "Datasheet" "http://www.njr.com/semicon/PDF/NJM5532_E.pdf" (id 3) (at 124.46 27.94 0)
       (effects (font (size 1.27 1.27)) hide)
     )
@@
       (effects (font (size 1.27 1.27)) hide)
     )
-    (property "Part Model No." "ALPS RK09L1240-F15-C0-A103(2連)" (id 4) (at 38.1 114.935 0)
+    (property "Part Model No." "ALPS RK09L1240-F15-C0-A103 2gang (2連)" (id 4) (at 38.1 114.935 0)
       (effects (font (size 1.27 1.27)) hide)
     )
@@
       (effects (font (size 1.27 1.27)) hide)
     )
-    (property "Part Model No." "サイズ max 5phi x 11mmまで" (id 4) (at 90.17 33.02 0)
+    (property "Part Model No." "サイズ max 5phi x 11mm" (id 4) (at 90.17 33.02 0)
       (effects (font (size 1.27 1.27)) hide)
     )
@@
     (pin "1")
   )
-  (symbol (lib_id "Amplifier_Operational:NJM4580") (at 150.495 27.94 0) (unit 3)
+  (symbol (lib_id "Amplifier_Operational:NJM5532") (at 150.495 27.94 0) (unit 3)
     (in_bom yes) (on_board yes)
     (property "Reference" "U2" (id 0) (at 149.479 26.6699 0)
@@
       (effects (font (size 1.27 1.27)) hide)
     )
-    (property "Datasheet" "http://www.njr.com/semicon/PDF/NJM4580_E.pdf" (id 3) (at 150.495 27.94 0)
+    (property "Datasheet" "http://www.njr.com/semicon/PDF/NJM5532_E.pdf" (id 3) (at 150.495 27.94 0)
       (effects (font (size 1.27 1.27)) hide)
     )
@@
       (effects (font (size 1.27 1.27)) hide)
     )
-    (property "Part Model No." "サイズ max 5phi x 11mmまで" (id 4) (at 40.64 73.025 0)
+    (property "Part Model No." "サイズ max 5phi x 11mm" (id 4) (at 40.64 73.025 0)
       (effects (font (size 1.27 1.27)) hide)
     )
@@
       (effects (font (size 1.27 1.27)) hide)
     )
-    (property "Part Model No." "サイズ max 5phi x 11mmまで" (id 4) (at 40.64 55.245 0)
+    (property "Part Model No." "サイズ max 5phi x 11mm" (id 4) (at 40.64 55.245 0)
       (effects (font (size 1.27 1.27)) hide)
     )
@@
       (effects (font (size 1.27 1.27)) hide)
     )
-    (property "Part Model No." "ALPS RK09L1240-F15-C0-B503(2連)" (id 4) (at 229.87 76.835 0)
+    (property "Part Model No." "ALPS RK09L1240-F15-C0-B503 2gang (2連)" (id 4) (at 229.87 76.835 0)
       (effects (font (size 1.27 1.27)) hide)
     )
@@
     (pin "1")
   )
-  (symbol (lib_id "Amplifier_Operational:NJM4580") (at 135.255 52.705 0) (unit 2)
+  (symbol (lib_id "Amplifier_Operational:NJM5532") (at 135.255 52.705 0) (unit 2)
     (in_bom yes) (on_board yes) (fields_autoplaced)
     (property "Reference" "U1" (id 0) (at 135.255 41.91 0))
@@
       (effects (font (size 1.27 1.27)) hide)
     )
-    (property "Datasheet" "http://www.njr.com/semicon/PDF/NJM4580_E.pdf" (id 3) (at 135.255 52.705 0)
+    (property "Datasheet" "http://www.njr.com/semicon/PDF/NJM5532_E.pdf" (id 3) (at 135.255 52.705 0)
       (effects (font (size 1.27 1.27)) hide)
     )
@@
       (effects (font (size 1.27 1.27)) hide)
     )
-    (property "Part Model No." "サイズ max 5phi x 11mmまで" (id 4) (at 43.18 108.585 0)
+    (property "Part Model No." "サイズ max 5phi x 11mm" (id 4) (at 43.18 108.585 0)
       (effects (font (size 1.27 1.27)) hide)
     )
@@
     (pin "2")
   )
-  (symbol (lib_id "Amplifier_Operational:NJM4580") (at 176.53 27.94 0) (unit 3)
+  (symbol (lib_id "Amplifier_Operational:NJM5532") (at 176.53 27.94 0) (unit 3)
     (in_bom yes) (on_board yes)
     (property "Reference" "U3" (id 0) (at 175.514 26.6699 0)
@@
       (effects (font (size 1.27 1.27)) hide)
     )
-    (property "Datasheet" "http://www.njr.com/semicon/PDF/NJM4580_E.pdf" (id 3) (at 176.53 27.94 0)
+    (property "Datasheet" "http://www.njr.com/semicon/PDF/NJM5532_E.pdf" (id 3) (at 176.53 27.94 0)
       (effects (font (size 1.27 1.27)) hide)
     )
@@
       (effects (font (size 1.27 1.27)) hide)
     )
-    (property "Part Model No." "サイズ max 5phi x 11mmまで" (id 4) (at 43.18 121.285 0)
+    (property "Part Model No." "サイズ max 5phi x 11mm" (id 4) (at 43.18 121.285 0)
       (effects (font (size 1.27 1.27)) hide)
     )
@@
       (effects (font (size 1.27 1.27)) hide)
     )
-    (property "Part Model No." "サイズ max 5phi x 11mmまで" (id 4) (at 40.005 150.495 0)
+    (property "Part Model No." "サイズ max 5phi x 11mm" (id 4) (at 40.005 150.495 0)
       (effects (font (size 1.27 1.27)) hide)
     )
@@
       (effects (font (size 1.27 1.27)) hide)
     )
-    (property "Part Model No." "サイズ max 5phi x 11mmまで" (id 4) (at 40.64 90.805 0)
+    (property "Part Model No." "サイズ max 5phi x 11mm" (id 4) (at 40.64 90.805 0)
       (effects (font (size 1.27 1.27)) hide)
     )
@@
       (effects (font (size 1.27 1.27)) hide)
     )
-    (property "Part Model No." "NKK B-12CCPRM" (id 4) (at 45.72 20.32 0)
+    (property "Part Model No." "NKK B-12CCPR" (id 4) (at 45.72 20.32 0)
       (effects (font (size 1.27 1.27)) hide)
     )
@@
       (effects (font (size 1.27 1.27)) hide)
     )
-    (property "Part Model No." "サイズ max 5phi x 11mmまで" (id 4) (at 146.05 147.955 0)
+    (property "Part Model No." "サイズ max 5phi x 11mm" (id 4) (at 146.05 147.955 0)
       (effects (font (size 1.27 1.27)) hide)
     )
@@
       (effects (font (size 1.27 1.27)) hide)
     )
-    (property "Part Model No." "サイズ max 5phi x 11mmまで" (id 4) (at 40.005 168.275 0)
+    (property "Part Model No." "サイズ max 5phi x 11mm" (id 4) (at 40.005 168.275 0)
       (effects (font (size 1.27 1.27)) hide)
     )
@@
       (effects (font (size 1.27 1.27)) hide)
     )
-    (property "Part Model No." "サイズ max 5phi x 11mmまで" (id 4) (at 146.685 52.705 0)
+    (property "Part Model No." "サイズ max 5phi x 11mm" (id 4) (at 146.685 52.705 0)
       (effects (font (size 1.27 1.27)) hide)
     )
@@
     (pin "2")
   )
-  (symbol (lib_id "Amplifier_Operational:NJM4580") (at 134.62 147.955 0) (unit 2)
+  (symbol (lib_id "Amplifier_Operational:NJM5532") (at 134.62 147.955 0) (unit 2)
     (in_bom yes) (on_board yes) (fields_autoplaced)
     (property "Reference" "U2" (id 0) (at 134.62 137.16 0))
@@
       (effects (font (size 1.27 1.27)) hide)
     )
-    (property "Datasheet" "http://www.njr.com/semicon/PDF/NJM4580_E.pdf" (id 3) (at 134.62 147.955 0)
-      (effects (font (size 1.27 1.27)) hide)
-    )
+    (property "Datasheet" "http://www.njr.com/semicon/PDF/NJM5532_E.pdf" (id 3) (at 134.62 147.955 0)
+      (effects (font (size 1.27 1.27)) hide)
+    )
